File: Internal Version/FDC.kicad_pcb (KiCad board)
At the start: 2 copper layers, 37.8 x 110.5 mm, 26 parts, among them J1 Conn_01x01_Pin, Q1 FDV301N, Q2 FDV301N, U1 SN74LVC245APWR, U10 Z80, U11 Z80, U2 SN74LVC245APWR, U3 SN74LVC245APWR, U4 SN74LVC245APWR, U5 SN74LS32NSR

Commit message: Updated silkscreen on gerbers
Other:
- board text added: "Floppy80-M1 ver 1.45 Internal version by dabone (2026) https://github.com/dabonetn/Floppy80-M1-Internal Original By MichaelM4 https://github.com/MichaelM4/Floppy80-M1"
- board text removed: "Floppy80-M1 ver 1.4 Internal version by dabone (2026) https://github.com/dabonetn/Floppy80-M1-Internal Original By MichaelM4 https://github.com/MichaelM4/Floppy80-M1"
Changed lines of the file:
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@@
 		)
 	)
-	(gr_text "Floppy80-M1 ver 1.4\nInternal version by dabone (2026)\nhttps://github.com/dabonetn/Floppy80-M1-Internal\nOriginal By MichaelM4\nhttps://github.com/MichaelM4/Floppy80-M1"
+	(gr_text "Floppy80-M1 ver 1.45\nInternal version by dabone (2026)\nhttps://github.com/dabonetn/Floppy80-M1-Internal\nOriginal By MichaelM4\nhttps://github.com/MichaelM4/Floppy80-M1"
 		(at 141.9 122.4 90)
 		(layer "B.SilkS")
@@
 	)
 	(segment
+		(start 135.37 42.075)
+		(end 133.425 42.075)
+		(width 0.4)
+		(layer "F.Cu")
+		(net "/5vPico")
+	)
+	(segment
+		(start 133.425 42.075)
+		(end 133.3 42.2)
+		(width 0.25)
+		(layer "F.Cu")
+		(net "/5vPico")
+	)
+	(via
+		(at 133.3 42.2)
+		(size 0.8)
+		(drill 0.4)
+		(layers "F.Cu" "B.Cu")
+		(net "/5vPico")
+	)
+	(segment
+		(start 137.035 43.435)
+		(end 137.3823 43.7823)
+		(width 0.25)
+		(layer "B.Cu")
+		(net "/5vPico")
+	)
+	(segment
+		(start 137.035 43.435)
+		(end 134.535 43.435)
+		(width 0.4)
+		(layer "B.Cu")
+		(net "/5vPico")
+	)
+	(segment
+		(start 134.535 43.435)
+		(end 133.3 42.2)
+		(width 0.4)
+		(layer "B.Cu")
+		(net "/5vPico")
+	)
+	(segment
 		(start 153.125 120.925)
 		(end 152.3904 120.925)
@@
 		(net "/INT'")
 	)
-	(segment
-		(start 135.37 42.075)
-		(end 133.425 42.075)
-		(width 0.4)
-		(layer "F.Cu")
-		(net "/5vPico")
-	)
-	(segment
-		(start 133.425 42.075)
-		(end 133.3 42.2)
-		(width 0.25)
-		(layer "F.Cu")
-		(net "/5vPico")
-	)
-	(via
-		(at 133.3 42.2)
-		(size 0.8)
-		(drill 0.4)
-		(layers "F.Cu" "B.Cu")
-		(net "/5vPico")
-	)
-	(segment
-		(start 137.035 43.435)
-		(end 137.3823 43.7823)
-		(width 0.25)
-		(layer "B.Cu")
-		(net "/5vPico")
-	)
-	(segment
-		(start 137.035 43.435)
-		(end 134.535 43.435)
-		(width 0.4)
-		(layer "B.Cu")
-		(net "/5vPico")
-	)
-	(segment
-		(start 134.535 43.435)
-		(end 133.3 42.2)
-		(width 0.4)
-		(layer "B.Cu")
-		(net "/5vPico")
-	)
 	(zone
